File: projects/adon/adon.kicad_pcb (KiCad board)
At the start: 2 copper layers, 55.9 x 30.5 mm, 29 parts, among them IC1 STM32F030F4, P1 BATTERY, P2 SWD, Q1 2N3704, SW1 POWER, SW2 BUTTON0, SW3 BUTTON1, SW4 BUTTON2, SW5 BUTTON3

Commit message: awh yeah
Parts:
- added D1: ERROR, LEDs:LED-0805, F.Cu at (31.5, 25.9)
- added R9: 330, Resistors_SMD:Resistor_SMD0805_HandSoldering_RevA_Date21Jun2010, F.Cu at (30.0, 29.5)
- JP1: footprint open-project:S_JUMPER_3 -> Connect:SIL-3
- SP1: footprint Buzzer:MagneticBuzzer_ProSignal_ABT-410-RC_RevA_25Oct2010 -> Buzzer:MagneticBuzzer_Kingstate_KCG0601_RevA_25Oct2010
- moved R5 107.3 mm to (17.8, 34.5), turned to 90 degrees
- moved R8 93.6 mm to (30.0, 32.5), turned to 180 degrees
- moved D6 83.6 mm to (26.9, 25.9)
- moved R7 75.6 mm to (43.2, 29.5)
- moved C4 71.0 mm to (48.8, 20.3), turned to 270 degrees
- moved C2 70.9 mm to (46.2, 20.3), turned to 90 degrees
- moved JP1 70.4 mm to (36.1, 17.3)
- moved IC1 66.1 mm to (54.4, 19.3), turned to 270 degrees
- moved Q1 65.4 mm to (34.0, 21.8), turned to 180 degrees
- moved C3 62.8 mm to (62.5, 20.3), turned to 270 degrees
- moved C1 62.4 mm to (22.9, 22.9), turned to 90 degrees
- moved R4 61.2 mm to (43.2, 32.5)
- moved R2 57.9 mm to (43.7, 19.8), turned to 270 degrees
- moved C5 57.0 mm to (59.9, 20.3), turned to 270 degrees
- moved R6 56.2 mm to (56.4, 29.5)
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Connections:
- JP1 pad 3: (no net) -> Net-(JP1-Pad2)
Other:
- board text added: "Adon v5 arolsen@gmail.com"

Commit message: woot
Parts:
- SP1: footprint Buzzer:MagneticBuzzer_Kingstate_KCG0601_RevA_25Oct2010 -> synic:Buzzer_CUI_INC_CC-1601
- moved R2 16.0 mm to (59.4, 22.4), turned to 180 degrees
- moved R8 13.6 mm to (20.3, 22.9), turned to 0 degrees
- moved SP1 9.43 mm to (37.1, 16.8), turned to 180 degrees
- moved D6 8.65 mm to (20.3, 20.3)
- moved C1 8.14 mm to (22.4, 14.7), turned to 0 degrees
- moved D1 7.55 mm to (26.4, 20.3), turned to 180 degrees
- moved JP1 7.55 mm to (29.0, 14.7), turned to 180 degrees
- moved R9 7.50 mm to (26.4, 22.9), turned to 0 degrees
- moved C2 5.92 mm to (43.2, 15.2), turned to 0 degrees
- moved C4 4.68 mm to (45.2, 17.3), turned to 180 degrees
- moved C5 3.21 mm to (58.9, 17.3), turned to 0 degrees
- moved SW3 2.87 mm to (34.5, 38.6)
- moved D4 2.87 mm to (34.5, 28.4)
- moved IC1 2.87 mm to (52.3, 17.3)
- moved Q1 2.87 mm to (32.0, 19.8)
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Routing:
- net Net-(IC1-Pad9): track 0.00 -> 52.3 mm
- net Net-(IC1-Pad13): track 0.00 -> 35.0 mm, vias 0 -> 1
- net Net-(IC1-Pad12): track 0.00 -> 34.7 mm, vias 0 -> 1
- net SWCLK: track 0.00 -> 20.2 mm
- net VDD: track 0.00 -> 19.0 mm
- net SWDIO: track 0.00 -> 18.1 mm
- net Net-(D2-Pad1): track 0.00 -> 8.75 mm
- net NRST: track 0.00 -> 7.18 mm
- net GND: track 0.00 -> 6.22 mm
- net (no net): track 0.00 -> 0.77 mm
- net Net-(D5-Pad1): track 0.00 -> 0.76 mm
- net Net-(D4-Pad1): track 0.00 -> 0.76 mm
- added copper zone on F.Cu, net GND
- added copper zone on B.Cu, net VDD

Commit message: woot
Parts:
- moved R1 26.4 mm to (27.9, 30.5)
- moved R6 26.4 mm to (27.9, 27.4), turned to 180 degrees
Routing:
- net VDD: track 19.0 -> 69.1 mm
- net Net-(D4-Pad1): track 0.76 -> 45.9 mm
- net GND: track 6.22 -> 46.5 mm
- net Net-(IC1-Pad10): track 0.00 -> 40.3 mm, vias 0 -> 1
- net Net-(IC1-Pad11): track 0.00 -> 38.6 mm, vias 0 -> 1
- net NRST: track 7.18 -> 41.1 mm, vias 0 -> 1
- net Net-(D1-Pad1): track 0.00 -> 33.4 mm, vias 0 -> 2
- net Net-(Q1-Pad3): track 0.00 -> 30.1 mm, vias 0 -> 2
- net Net-(IC1-Pad8): track 0.00 -> 29.5 mm, vias 0 -> 2
- net Net-(IC1-Pad18): track 0.00 -> 25.5 mm, vias 0 -> 1
- net Net-(P1-Pad1): track 0.00 -> 9.71 mm
- net Net-(JP1-Pad2): track 0.49 -> 7.88 mm
- net Net-(D5-Pad1): track 0.76 -> 7.42 mm
- net Net-(D3-Pad1): track 0.00 -> 4.88 mm
- net Net-(D6-Pad2): track 0.00 -> 3.51 mm
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
Commit message: done
Parts:
- C1: footprint Capacitors_SMD:c_1206 -> Capacitors_SMD:c_elec_5x5.3
- D1: value ERROR -> FAIL
- moved R3 12.3 mm to (54.5, 30.4), turned to 180 degrees
- moved R2 7.06 mm to (54.5, 27.4)
- moved C2 3.92 mm to (44.6, 18.9), turned to 90 degrees
- moved C1 3.85 mm to (25.1, 17.4), turned to 270 degrees
- moved R9 3.61 mm to (30.0, 22.4)
- moved D1 3.58 mm to (30.0, 19.9)
- moved JP1 3.35 mm to (32.3, 14.8)
- moved C4 3.03 mm to (47.4, 19.3), turned to 270 degrees
- moved SP1 2.54 mm to (39.6, 17.2)
- moved C5 1.98 mm to (60.8, 18.0), turned to 90 degrees
- moved Q1 1.78 mm to (33.6, 19.1)
- moved IC1 1.67 mm to (54.0, 17.3)
- moved R8 0.57 mm to (20.1, 22.4), turned to 180 degrees
- moved D6 0.46 mm to (20.1, 19.9)
Routing:
- net Net-(IC1-Pad7): track 0.00 -> 44.9 mm
- net Net-(IC1-Pad9): track 52.3 -> 13.3 mm
- net VDD: track 69.1 -> 104.1 mm, vias 0 -> 2
- net GND: track 46.5 -> 81.3 mm, vias 0 -> 3
- net Net-(IC1-Pad1): track 0.00 -> 32.8 mm
- net Net-(IC1-Pad6): track 0.00 -> 30.8 mm, vias 0 -> 2
- net Net-(D4-Pad1): track 45.9 -> 18.9 mm
- net NRST: track 41.1 -> 24.4 mm, vias 1 -> 0
- net Net-(IC1-Pad8): track 29.5 -> 18.7 mm, vias 2 -> 0
- net Net-(Q1-Pad3): track 30.1 -> 19.7 mm, vias 2 -> 1
- net SWDIO: track 18.1 -> 24.3 mm
- net SWCLK: track 20.2 -> 14.8 mm
- net Net-(IC1-Pad13): track 35.5 -> 40.5 mm, vias 1 -> 0
- net Net-(IC1-Pad10): track 40.3 -> 44.0 mm, vias 1 -> 0
- net Net-(IC1-Pad18): track 25.5 -> 22.4 mm
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- added copper zone on B.Cu, net GND

Commit message: tssop bitches
Parts:
- D1: value FAIL -> ERROR
- IC1: footprint synic:tssop-20 -> ab2:AB2_TSSOP20
- moved R5 48.7 mm to (61.2, 15.1), turned to 180 degrees
- moved IC1 3.03 mm to (54.0, 20.4)
- moved C5 2.47 mm to (60.2, 20.5)
- moved C3 1.90 mm to (62.6, 20.4), turned to 90 degrees
- moved C2 1.85 mm to (45.6, 20.4)
- moved C4 1.20 mm to (47.9, 20.4)
- moved SP1 0.12 mm to (39.6, 17.3)
Routing:
- net VDD: track 104.1 -> 0.00 mm, vias 2 -> 0
- net GND: track 81.3 -> 0.00 mm, vias 3 -> 0
- net Net-(IC1-Pad7): track 44.9 -> 0.00 mm
- net Net-(IC1-Pad10): track 44.0 -> 0.00 mm
- net Net-(IC1-Pad13): track 40.5 -> 0.00 mm
- net Net-(IC1-Pad11): track 38.9 -> 0.00 mm, vias 1 -> 0
- net Net-(IC1-Pad12): track 33.7 -> 0.00 mm, vias 1 -> 0
- net Net-(IC1-Pad1): track 32.8 -> 0.00 mm
- net Net-(D1-Pad1): track 31.1 -> 0.00 mm
- net Net-(IC1-Pad6): track 30.8 -> 0.00 mm, vias 2 -> 0
- net NRST: track 24.4 -> 0.00 mm
- net SWDIO: track 24.3 -> 0.00 mm
- net Net-(IC1-Pad18): track 22.4 -> 0.00 mm, vias 1 -> 0
- net Net-(Q1-Pad3): track 19.7 -> 0.00 mm, vias 1 -> 0
- net Net-(D4-Pad1): track 18.9 -> 0.00 mm
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- removed copper zone on B.Cu, net VDD
Other:
- board text removed: "Adon v5 arolsen@gmail.com"

Commit message: woot
Routing:
- net VDD: track 0.00 -> 180.5 mm, vias 0 -> 1
- net GND: track 0.00 -> 77.5 mm, vias 0 -> 4
- net Net-(IC1-Pad10): track 0.00 -> 43.1 mm
- net Net-(IC1-Pad13): track 0.00 -> 37.0 mm
- net Net-(IC1-Pad11): track 0.00 -> 34.3 mm, vias 0 -> 1
- net Net-(D4-Pad1): track 0.00 -> 33.0 mm, vias 0 -> 1
- net Net-(IC1-Pad1): track 0.00 -> 32.6 mm
- net Net-(D1-Pad1): track 0.00 -> 30.9 mm
- net Net-(IC1-Pad12): track 0.00 -> 30.6 mm, vias 0 -> 1
- net Net-(IC1-Pad6): track 0.00 -> 26.2 mm, vias 0 -> 2
- net SWDIO: track 0.00 -> 25.6 mm
- net Net-(IC1-Pad18): track 0.00 -> 23.6 mm
- net NRST: track 0.00 -> 21.8 mm
- net Net-(Q1-Pad3): track 0.00 -> 17.6 mm, vias 0 -> 1
- net Net-(IC1-Pad8): track 0.00 -> 15.4 mm
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
Commit message: woot
Parts:
- turned C3 to 270 degrees
- turned C5 to 270 degrees
Routing:
- net GND: track 77.5 -> 69.4 mm, vias 4 -> 3
- net Net-(IC1-Pad13): track 37.0 -> 39.0 mm
- net VDD: track 180.5 -> 179.4 mm

Commit message: woooo!
Routing:
- net GND: track 69.4 -> 87.3 mm, vias 3 -> 5
- net Net-(IC1-Pad6): track 26.2 -> 25.5 mm
Changed lines of the file:
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@@
   (general
     (links 65)
-    (no_connects 3)
+    (no_connects 0)
     (area 13.157999 13.157999 69.138001 43.738001)
     (thickness 1.6)
     (drawings 4)
-    (tracks 252)
+    (tracks 266)
     (zones 0)
     (modules 31)
@@
   (gr_line (start 13.208 43.688) (end 69.088 43.688) (angle 90) (layer Edge.Cuts) (width 0.1))
   (gr_line (start 13.208 13.208) (end 13.208 43.688) (angle 90) (layer Edge.Cuts) (width 0.1))
-  (segment (start 62.5729 19.4945) (end 65.278 19.4945) (width 0.254) (layer F.Cu) (net 1) (status 400000))
-  (segment (start 67.6656 16.6116) (end 66.548 15.494) (width 0.254) (layer F.Cu) (net 1) (status 800000))
+  (segment (start 62.5729 19.4945) (end 65.278 19.4945) (width 0.254) (layer F.Cu) (net 1))
+  (segment (start 67.6656 16.6116) (end 66.548 15.494) (width 0.254) (layer F.Cu) (net 1))
   (segment (start 67.6656 18.780298) (end 67.6656 16.6116) (width 0.254) (layer F.Cu) (net 1))
   (segment (start 67.103798 19.3421) (end 67.6656 18.780298) (width 0.254) (layer F.Cu) (net 1))
@@
   (segment (start 34.9568 36.068) (end 34.9568 39.2999) (width 0.254) (layer B.Cu) (net 1))
   (segment (start 60.2488 19.4945) (end 60.2361 19.5072) (width 0.254) (layer F.Cu) (net 1))
-  (segment (start 60.2361 21.4122) (end 59.1312 21.4122) (width 0.254) (layer F.Cu) (net 2) (status 400000))
-  (segment (start 58.4148 20.6958) (end 56.8004 20.6958) (width 0.254) (layer F.Cu) (net 2) (status 800000))
+  (segment (start 62.23 28.448) (end 62.23 23.3045) (width 0.254) (layer B.Cu) (net 2))
+  (segment (start 62.5729 22.86) (end 62.5729 21.3995) (width 0.254) (layer F.Cu) (net 2))
+  (segment (start 62.1792 23.2537) (end 62.5729 22.86) (width 0.254) (layer F.Cu) (net 2))
+  (via (at 62.1792 23.2537) (size 0.889) (layers F.Cu B.Cu) (net 2))
+  (segment (start 62.23 23.3045) (end 62.1792 23.2537) (width 0.254) (layer B.Cu) (net 2))
+  (segment (start 45.593 21.3995) (end 47.879 21.3995) (width 0.254) (layer F.Cu) (net 2))
+  (segment (start 49.022 28.448) (end 49.022 25.5778) (width 0.254) (layer B.Cu) (net 2))
+  (segment (start 47.879 22.3012) (end 47.879 21.3995) (width 0.254) (layer F.Cu) (net 2))
+  (segment (start 46.8122 23.368) (end 47.879 22.3012) (width 0.254) (layer F.Cu) (net 2))
+  (via (at 46.8122 23.368) (size 0.889) (layers F.Cu B.Cu) (net 2))
+  (segment (start 49.022 25.5778) (end 46.8122 23.368) (width 0.254) (layer B.Cu) (net 2))
+  (segment (start 60.2361 21.4122) (end 59.1312 21.4122) (width 0.254) (layer F.Cu) (net 2))
+  (segment (start 58.4148 20.6958) (end 56.8004 20.6958) (width 0.254) (layer F.Cu) (net 2))
   (segment (start 59.1312 21.4122) (end 58.4148 20.6958) (width 0.254) (layer F.Cu) (net 2))
-  (segment (start 62.5729 21.3995) (end 60.2488 21.3995) (width 0.254) (layer F.Cu) (net 2) (status C00000))
-  (segment (start 60.2488 21.3995) (end 60.2361 21.4122) (width 0.254) (layer F.Cu) (net 2) (status C00000))
-  (segment (start 66.548 20.574) (end 64.4144 20.574) (width 0.254) (layer F.Cu) (net 2) (status 400000))
-  (segment (start 63.5889 21.3995) (end 62.5729 21.3995) (width 0.254) (layer F.Cu) (net 2) (status 800000))
+  (segment (start 62.5729 21.3995) (end 60.2488 21.3995) (width 0.254) (layer F.Cu) (net 2))
+  (segment (start 60.2488 21.3995) (end 60.2361 21.4122) (width 0.254) (layer F.Cu) (net 2))
+  (segment (start 66.548 20.574) (end 64.4144 20.574) (width 0.254) (layer F.Cu) (net 2))
+  (segment (start 63.5889 21.3995) (end 62.5729 21.3995) (width 0.254) (layer F.Cu) (net 2))
   (segment (start 64.4144 20.574) (end 63.5889 21.3995) (width 0.254) (layer F.Cu) (net 2))
   (segment (start 60.1218 21.4122) (end 60.2361 21.4122) (width 0.254) (layer F.Cu) (net 2))
@@
   (segment (start 21.3665 21.3713) (end 21.115 21.1198) (width 0.254) (layer F.Cu) (net 7))
   (segment (start 21.3665 22.352) (end 21.3665 21.3713) (width 0.254) (layer F.Cu) (net 7))
-  (via (at 44.1417 21.3786) (size 0.889) (layers F.Cu B.Cu) (net 8))
-  (via (at 37.2555 27.1172) (size 0.889) (layers F.Cu B.Cu) (net 8))
-  (segment (start 44.1417 21.9275) (end 44.1417 21.3786) (width 0.254) (layer F.Cu) (net 8))
-  (segment (start 44.6453 22.4311) (end 44.1417 21.9275) (width 0.254) (layer F.Cu) (net 8))
-  (segment (start 48.8002 22.4311) (end 44.6453 22.4311) (width 0.254) (layer F.Cu) (net 8))
-  (segment (start 50.0191 21.2122) (end 48.8002 22.4311) (width 0.254) (layer F.Cu) (net 8))
-  (segment (start 50.0191 20.6958) (end 50.0191 21.2122) (width 0.254) (layer F.Cu) (net 8))
-  (segment (start 38.4031 27.1172) (end 37.2555 27.1172) (width 0.254) (layer B.Cu) (net 8))
-  (segment (start 44.1417 21.3786) (end 38.4031 27.1172) (width 0.254) (layer B.Cu) (net 8))
-  (segment (start 30.6872 27.1172) (end 30.3724 27.432) (width 0.254) (layer F.Cu) (net 8))
-  (segment (start 37.2555 27.1172) (end 30.6872 27.1172) (width 0.254) (layer F.Cu) (net 8))
-  (segment (start 29.2405 27.432) (end 30.3724 27.432) (width 0.254) (layer F.Cu) (net 8))
-  (segment (start 51.2004 20.6958) (end 50.0191 20.6958) (width 0.254) (layer F.Cu) (net 8))
+  (segment (start 51.2004 20.6958) (end 49.6368 20.6958) (width 0.254) (layer F.Cu) (net 8))
+  (segment (start 30.51048 26.162) (end 29.24048 27.432) (width 0.254) (layer F.Cu) (net 8))
+  (segment (start 36.9062 26.162) (end 30.51048 26.162) (width 0.254) (layer F.Cu) (net 8))
+  (segment (start 37.4904 25.5778) (end 36.9062 26.162) (width 0.254) (layer F.Cu) (net 8))
+  (via (at 37.4904 25.5778) (size 0.889) (layers F.Cu B.Cu) (net 8))
+  (segment (start 43.815 25.5778) (end 37.4904 25.5778) (width 0.254) (layer B.Cu) (net 8))
+  (segment (start 44.1198 25.273) (end 43.815 25.5778) (width 0.254) (layer B.Cu) (net 8))
+  (via (at 44.1198 25.273) (size 0.889) (layers F.Cu B.Cu) (net 8))
+  (segment (start 46.3042 25.273) (end 44.1198 25.273) (width 0.254) (layer F.Cu) (net 8))
+  (segment (start 49.145388 22.431812) (end 46.3042 25.273) (width 0.254) (layer F.Cu) (net 8))
+  (segment (start 49.145388 21.187212) (end 49.145388 22.431812) (width 0.254) (layer F.Cu) (net 8))
+  (segment (start 49.6368 20.6958) (end 49.145388 21.187212) (width 0.254) (layer F.Cu) (net 8))
   (via (at 53.0596 20.9716) (size 0.889) (layers F.Cu B.Cu) (net 9))
   (via (at 61.9646 16.5156) (size 0.889) (layers F.Cu B.Cu) (net 9))
@@
   (segment (start 61.9646 16.5156) (end 62.3865 16.0937) (width 0.254) (layer F.Cu) (net 9))
   (segment (start 62.5145 15.113) (end 62.5145 16.0937) (width 0.254) (layer F.Cu) (net 9))
-  (segment (start 42.5156 29.4993) (end 39.8475 29.4993) (width 0.254) (layer F.Cu) (net 10))
-  (segment (start 50.0191 21.9958) (end 42.5156 29.4993) (width 0.254) (layer F.Cu) (net 10))
-  (segment (start 51.2004 21.9958) (end 50.0191 21.9958) (width 0.254) (layer F.Cu) (net 10))
-  (segment (start 39.8475 30.48) (end 39.8475 29.4993) (width 0.254) (layer F.Cu) (net 10))
+  (segment (start 51.2004 21.9958) (end 49.8862 21.9958) (width 0.254) (layer F.Cu) (net 10))
+  (segment (start 41.14292 29.1846) (end 39.84752 30.48) (width 0.254) (layer F.Cu) (net 10))
+  (segment (start 44.196 29.1846) (end 41.14292 29.1846) (width 0.254) (layer F.Cu) (net 10))
+  (segment (start 44.2722 29.1084) (end 44.196 29.1846) (width 0.254) (layer F.Cu) (net 10))
+  (segment (start 44.2722 28.0924) (end 44.2722 29.1084) (width 0.254) (layer F.Cu) (net 10))
+  (segment (start 49.657 22.7076) (end 44.2722 28.0924) (width 0.254) (layer F.Cu) (net 10))
+  (segment (start 49.657 22.225) (end 49.657 22.7076) (width 0.254) (layer F.Cu) (net 10))
+  (segment (start 49.8862 21.9958) (end 49.657 22.225) (width 0.254) (layer F.Cu) (net 10))
   (segment (start 68.196 21.466) (end 66.548 23.114) (width 0.254) (layer F.Cu) (net 11))
   (segment (start 68.196 15.2014) (end 68.196 21.466) (width 0.254) (layer F.Cu) (net 11))
